File: PCB's/Winder Core Board/Winder Core Board.kicad_sch (KiCad schematic)
At the start: 15 parts, among them J1 Speed_Pot, J2 Optical_Gate, J3 Conn_01x06_Pin, J4 Conn_01x06_Pin

Commit message: PCB updated. moved some pins.
Parts:
- removed RV1: R_Potentiometer, symbol Device:R_Potentiometer
- removed Tensioner_Port: Conn_01x04_Pin, symbol Connector:Conn_01x04_Pin
- added J5: Voltage Selector, Connector_JST:JST_EH_B3B-EH-A_1x03_P2.50mm_Vertical, symbol Connector:Conn_01x03_Socket
- added J6: Conn_01x02_Pin, Connector_JST:JST_EH_B2B-EH-A_1x02_P2.50mm_Vertical, symbol Connector:Conn_01x02_Pin
- added J7: SD_card EXT, Connector_JST:JST_EH_B6B-EH-A_1x06_P2.50mm_Vertical, symbol Connector:Conn_01x06_Socket
- added J8: Reset SW, Connector_JST:JST_EH_B2B-EH-A_1x02_P2.50mm_Vertical, symbol Connector:Conn_01x02_Pin
- added R_Serial1: 1k, Resistor_THT:R_Axial_DIN0207_L6.3mm_D2.5mm_P7.62mm_Horizontal, symbol Device:R
- C1: footprint (none) -> Capacitor_THT:CP_Radial_D8.0mm_P5.00mm
- HX711: renamed from U6; footprint (none) -> Connector_JST:JST_EH_B4B-EH-A_1x04_P2.50mm_Vertical
- J1, J2: footprint (none) -> Connector_JST:JST_EH_B3B-EH-A_1x03_P2.50mm_Vertical
- J3, J4: footprint (none) -> Connector_JST:JST_EH_B6B-EH-A_1x06_P2.50mm_Vertical
- Spindle_Port1: renamed from Spindle_Port; footprint (none) -> Connector_JST:JST_EH_B4B-EH-A_1x04_P2.50mm_Vertical
- Traverse_Port1: renamed from Traverse_Port; footprint (none) -> Connector_JST:JST_EH_B4B-EH-A_1x04_P2.50mm_Vertical
- U1, U3: footprint (none) -> CustomParts:TC2209
- U2: footprint (none) -> CustomParts:S3 DEvkit DualW
- U4: footprint (none) -> CustomParts:MS1584_fullboard
- U5: footprint (none) -> Connector_JST:JST_EH_B14B-EH-A_1x14_P2.50mm_Vertical
Connections:
- net +24V: now also U1.11 (V_mot), U3.11 (V_mot), J6.2 (Pin_2)
- net +3V3: now also J1.1 (Pin_1), J2.1 (Pin_1), J3.1 (Pin_1), J3.4 (Pin_4), J4.1 (Pin_1), J4.4 (Pin_4), J5.1 (Pin_1), J7.5 (Pin_5); no longer U4.3 (out+)
- net GND: now also J1.3 (Pin_3), J2.3 (Pin_3), J3.3 (Pin_3), J3.6 (Pin_6), J4.3 (Pin_3), J4.6 (Pin_6), U1.18 (GND), U3.18 (GND), J6.1 (Pin_1), J7.6 (Pin_6), J8.1 (Pin_1)
- net P1: now reaches U1.1 (EN)
- net P1: now also U2.26 (GPIO1)
- net at U1.13 (A2): now also Spindle_Port1.4 (Pin_4)
- net at U1.14 (A1): now also Spindle_Port1.3 (Pin_3)
- net at U1.15 (B1): now also Spindle_Port1.2 (Pin_2)
- net at U1.16 (B2): now also Spindle_Port1.1 (Pin_1)
- net at U1.2 (MS1): now also J4.2 (Pin_2)
- net at U1.3 (MS2): now also J4.5 (Pin_5)
- net P40: now reaches U1.4 (PDN_d)
- net P40: now also U2.30 (GPIO40), U3.4 (PDN_d), R_Serial1.1
- net P2: now reaches U1.7 (STEP)
- net P2: now also U2.27 (GPIO2), U2.29 (GPIO41)
- net P42: now reaches U1.8 (DIR)
- net P42: now also U2.28 (GPIO42)
- net P21: now reaches J2.2 (Pin_2)
- net P21: now also U2.40 (GPIO21)
- net P3: now reaches HX711.2 (DT)
- net P3: now also U2.13 (GPIO3)
- net P8: now reaches HX711.3 (SCK)
- net P8: now also U2.12 (GPIO8)
- net P14: now reaches J1.2 (Pin_2)
- net P14: now also U2.20 (GPIO14)
- net P36: now reaches U3.1 (EN)
- net P36: now also U2.35 (GPIO35)
- net at U3.13 (A2): now also Traverse_Port1.4 (Pin_4)
- net at U3.14 (A1): now also Traverse_Port1.3 (Pin_3)
- net at U3.15 (B1): now also Traverse_Port1.2 (Pin_2)
- net at U3.16 (B2): now also Traverse_Port1.1 (Pin_1)
- net at U3.2 (MS1): now also J3.2 (Pin_2)
- net at U3.3 (MS2): now also J3.5 (Pin_5)
- net P35: now reaches U3.7 (STEP)
- net P35: now also U2.32 (GPIO38), U2.34 (GPIO36)
- net P37: now reaches U3.8 (DIR)
- net P37: now also U2.33 (GPIO37)
- net P4: now reaches U5.1 (T_IRQ)
- net P4: now also U2.4 (GPIO4)
- net P16: now reaches U5.10 (DC)
- net P16: now also U2.9 (GPIO16)
- net P17: now reaches U5.11 (RESET)
- net P17: now also U2.10 (GPIO17)
- net P18: now reaches U5.12 (CS)
- net P18: now also U2.11 (GPIO18)
- net P5: now reaches U5.2 (T_DO)
- net P5: now also U2.5 (GPIO5), U5.6 (SDO(MISO))
- net P6: now reaches U5.3 (T_DIN)
- net P6: now also U2.6 (GPIO6), U5.9 (SDI(MOSI))
- net P7: now reaches U5.4 (T_CS)
- net P7: now also U2.7 (GPIO7)
- net P15: now reaches U5.5 (T_CLK)
- net P15: now also U2.8 (GPIO15), U5.8 (SCK)
- net P46: now reaches U2.14 (GPIO46)
- net P9: now reaches U2.15 (GPIO9)
- net P10: now reaches U2.16 (GPIO10)
- net P10: now also J7.1 (Pin_1)
- net P11: now reaches U2.17 (GPIO11)
- net P11: now also J7.3 (Pin_3)
- net P12: now reaches U2.18 (GPIO12)
- net P12: now also J7.2 (Pin_2)
- net P13: now reaches U2.19 (GPIO13)
- net P13: now also J7.4 (Pin_4)
- net 5V: now reaches U2.21 (5V0)
- net 5V: now also J5.3 (Pin_3)
- net RST: now reaches U2.3 (RST)
- net RST: now also J8.2 (Pin_2)
- net P39: now reaches U2.31 (GPIO39)
- net P39: now also R_Serial1.2
- net P0: now reaches U2.36 (GPIO0)
- net P45: now reaches U2.37 (GPIO45)
- net P48: now reaches U2.38 (GPIO48)
- net P47: now reaches U2.39 (GPIO47)
- net P20: now reaches U2.41 (GPIO20)
- net P19: now reaches U2.42 (GPIO19)
- new net: J5.2 (Pin_2), U4.3 (out+)
Other:
- moved on the sheet: HX711, J1, J2, J3, J4, Spindle_Port1, Traverse_Port1, U2, U5
